File: circuit/fortuna-5.kicad_sch (KiCad schematic)
At the start: 13 parts, among them J8 USB-C Power, SW1 SW_Push, SW4 SW_DPDT_x2, U1 ATmega2560-16C, U2 Z80CPU, U3 AS6C4008-55PCN, U4 74HC04, U5 74LS32, U6 74HC00

Commit message: .
Connections:
- net SCLK is gone; now on net SIMCLK: SW4.3 (C)
- net A0: now also U1.A3 (PF0), U2.30 (A0), U3.12 (A0)
- net A1: now also U1.B3 (PF1), U2.31 (A1), U3.11 (A1)
- net A10: now also U1.C6 (PK2), U2.40 (A10), U3.23 (A10)
- net A11: now also U1.A7 (PK3), U2.1 (A11), U3.25 (A11)
- net A12: now also U1.B7 (PK4), U2.2 (A12), U3.4 (A12)
- net A13: now also U1.C7 (PK5), U2.3 (A13), U3.28 (A13)
- net A14: now also U1.A8 (PK6), U2.4 (A14), U3.3 (A14)
- net A15: now also U1.B8 (PK7), U2.5 (A15), U3.31 (A15)
- net A16: now also U1.G5 (PL2), U3.2 (A16)
- net A17: now also U1.H5 (PL3), U3.30 (A17)
- net A18: now also U1.K6 (PL5), U3.1 (A18)
- net A2: now also U1.A4 (PF2), U2.32 (A2), U3.10 (A2)
- net A3: now also U1.B4 (PF3), U2.33 (A3), U3.9 (A3)
- net A4: now also U1.C4 (PF4), U2.34 (A4), U3.8 (A4)
- net A5: now also U1.A5 (PF5), U2.35 (A5), U3.7 (A5)
- net A6: now also U1.B5 (PF6), U2.36 (A6), U3.6 (A6)
- net A7: now also U1.C5 (PF7), U2.37 (A7), U3.5 (A7)
- net A8: now also U1.A6 (PK0), U2.38 (A8), U3.27 (A8)
- net A9: now also U1.B6 (PK1), U2.39 (A9), U3.26 (A9)
- net D0: now also U1.B9 (PA0), U2.14 (D0), U3.13 (DQ0)
- net D1: now also U1.C9 (PA1), U2.15 (D1), U3.14 (DQ1)
- net D2: now also U1.B10 (PA2), U2.12 (D2), U3.15 (DQ2)
- net D3: now also U1.C10 (PA3), U2.8 (D3), U3.17 (DQ3)
- net D4: now also U1.D6 (PA4), U2.7 (D4), U3.18 (DQ4)
- net D5: now also U1.D7 (PA5), U2.9 (D5), U3.19 (DQ5)
- net D6: now also U1.D8 (PA6), U2.10 (D6), U3.20 (DQ6)
- net D7: now also U1.D9 (PA7), U2.13 (D7), U3.21 (DQ7)
- net GND: now also U1.A1 (GND), U1.A9 (GND), U1.F10 (GND), U1.G1 (GND), U1.K4 (GND), U2.29 (GND), U3.16 (VSS)
- net VCC: now also U1.A10 (VCC), U1.F1 (VCC), U1.G10 (VCC), U1.K3 (VCC), U2.11 (VCC), U3.32 (VCC)
- net ZCLK: now also U2.6 (~{CLK})
- net ~{BUSAK}: now also U1.E2 (PH0), U2.23 (~{BUSACK})
- net ~{BUSRQ}: now also U1.G8 (PC5), U2.25 (~{BUSRQ})
- net ~{CWAIT}: now also U1.G9 (PC6)
- net ~{INT}: now also U1.J8 (PC1), U2.16 (~{INT})
- net ~{IORQ}: now also U1.G6 (PD0), U2.20 (~{IORQ})
- net ~{M1}: now also U1.F6 (PD1), U2.27 (~{M1})
- net ~{MREQ}: now also U1.H8 (PC4), U2.19 (~{MREQ}), U3.22 (CE#)
- net ~{NMI}: now also U1.J9 (PC0), U2.17 (~{NMI})
- net ~{RD}: now also U1.H10 (PC2), U2.21 (~{RD}), U3.24 (OE#)
- net ~{SCLK_ENA}: now also U1.D10 (PG2)
- net ~{WAIT}: now also U1.K7 (PD2), U2.24 (~{WAIT})
- net ~{WR}: now also U1.H9 (PC3), U2.22 (~{WR}), U3.29 (WE#)
- net ~{HALT}: now reaches U2.18 (~{HALT})
- net ~{HALT}: now also U1.J7 (PD3)
- net ~{RESET}: now reaches U2.26 (~{RESET})
- net ~{RESET}: now also U1.H6 (PL7)
- net ~{CS0}: now reaches U1.F4 (PB0)
- net SCK: now reaches U1.G2 (PB1)
- net MOSI: now reaches U1.G3 (PB2)
- net ~{CS2}: now reaches U1.G4 (PB5)
- net MISO: now reaches U1.H1 (PB3)
- net ~{CS1}: now reaches U1.H2 (PB4)
- net SIMCLK: now reaches U1.H4 (PL1)
- no-connect marks 25 -> 26
Other:
- note added: "CPU"
- note added: "Debugger / IO"
- note added: "RAM"
- moved on the sheet: U1, U2, U3

Commit message: .
Connections:
- net ~{NMI}: now also U1.K10 (PG0); no longer U1.J9 (PC0)
Changed lines of the file:
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@@
-    (stroke (width 0) (type default))
-  )
-  (wire (pts (xy 76.2 88.265) (xy 86.36 88.265))
     (stroke (width 0) (type default))
   )
@@
   )
   (wire (pts (xy 153.67 50.165) (xy 163.83 50.165))
+    (stroke (width 0) (type default))
+  )
+  (wire (pts (xy 35.56 156.845) (xy 25.4 156.845))
     (stroke (width 0) (type default))
   )
@@
     (effects (font (size 1.27 1.27)) (justify left bottom))
   )
-  (label "~{NMI}" (at 86.36 88.265 180) (fields_autoplaced)
-    (effects (font (size 1.27 1.27)) (justify right bottom))
-  )
   (label "A13" (at -205.105 163.83 0) (fields_autoplaced)
     (effects (font (size 1.27 1.27)) (justify left bottom))
@@
     (effects (font (size 1.27 1.27)) (justify left bottom))
   )
+  (label "~{NMI}" (at 25.4 156.845 0) (fields_autoplaced)
+    (effects (font (size 1.27 1.27)) (justify left bottom))
+  )

Commit message: .
Connections:
- net ~{CWAIT}: now also U1.F8 (PJ0); no longer U1.G9 (PC6)
Changed lines of the file:
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@@
-    (stroke (width 0) (type default))
-  )
-  (wire (pts (xy 76.2 103.505) (xy 86.36 103.505))
     (stroke (width 0) (type default))
   )
@@
   )
   (wire (pts (xy 189.23 46.355) (xy 179.07 46.355))
+    (stroke (width 0) (type default))
+  )
+  (wire (pts (xy 35.56 111.125) (xy 25.4 111.125))
     (stroke (width 0) (type default))
   )
@@
     (effects (font (size 1.27 1.27)) (justify right bottom))
   )
+  (label "~{CWAIT}" (at 25.4 111.125 0) (fields_autoplaced)
+    (effects (font (size 1.27 1.27)) (justify left bottom))
+  )
   (label "D1" (at 86.36 45.085 180) (fields_autoplaced)
     (effects (font (size 1.27 1.27)) (justify right bottom))
@@
     (effects (font (size 1.27 1.27)) (justify right bottom))
   )
-  (label "~{CWAIT}" (at 86.36 103.505 180) (fields_autoplaced)
-    (effects (font (size 1.27 1.27)) (justify right bottom))
-  )

Commit message: .
Parts:
- added D2: CLOCK, symbol Device:LED
- added R1: R, symbol Device:R
- SW1, SW4: value SW_DPDT_x2 -> CLOCK
Connections:
- net GND: now also SW1.4 (A), R1.2; no longer SW1.6 (C)
- net SIMCLK: now also SW4.1 (A); no longer SW4.3 (C)
- net VCC: no longer SW1.4 (A)
- net ~{SCLK_ENA}: now also U1.J3 (PB6); no longer U1.D10 (PG2)
- net at U1.F3 (PH6): now also D2.2 (A)
- net at X?.8 (OUT): now also SW4.3 (C); no longer SW4.1 (A)
- new net: D2.1 (K), R1.1
- no-connect marks 26 -> 27
Other:
- moved on the sheet: SW1B, SW4A
Changed lines of the file:
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@@
   (no_connect (at -194.31 184.15))
   (no_connect (at -194.31 201.93))
+  (no_connect (at 257.81 146.05))
   (no_connect (at -194.31 105.41))
   (no_connect (at -162.56 86.36))
@@
     (stroke (width 0) (type default))
   )
+  (wire (pts (xy 14.605 152.4) (xy 14.605 149.225))
+    (stroke (width 0) (type default))
+  )
   (wire (pts (xy -216.535 179.705) (xy -216.535 176.53))
     (stroke (width 0) (type default))
@@
     (stroke (width 0) (type default))
   )
-  (wire (pts (xy 270.51 147.32) (xy 267.97 147.32))
-    (stroke (width 0) (type default))
-  )
   (wire (pts (xy -117.475 143.51) (xy -128.27 143.51))
     (stroke (width 0) (type default))
@@
     (stroke (width 0) (type default))
   )
+  (wire (pts (xy 14.605 160.02) (xy 14.605 161.29))
+    (stroke (width 0) (type default))
+  )
   (wire (pts (xy 153.67 45.085) (xy 163.83 45.085))
     (stroke (width 0) (type default))
@@
     (stroke (width 0) (type default))
   )
-  (wire (pts (xy 270.51 152.4) (xy 270.51 154.94))
+  (wire (pts (xy 255.27 151.13) (xy 255.27 153.67))
     (stroke (width 0) (type default))
   )
@@
     (stroke (width 0) (type default))
   )
+  (wire (pts (xy 86.36 80.645) (xy 76.2 80.645))
+    (stroke (width 0) (type default))
+  )
   (wire (pts (xy 135.89 111.125) (xy 135.89 114.935))
     (stroke (width 0) (type default))
@@
     (stroke (width 0) (type default))
   )
-  (wire (pts (xy 270.51 144.78) (xy 270.51 147.32))
-    (stroke (width 0) (type default))
-  )
-  (wire (pts (xy 245.11 149.86) (xy 257.81 149.86))
+  (wire (pts (xy 280.67 148.59) (xy 267.97 148.59))
     (stroke (width 0) (type default))
   )
@@
     (stroke (width 0) (type default))
   )
-  (wire (pts (xy 22.86 161.925) (xy 35.56 161.925))
-    (stroke (width 0) (type default))
-  )
   (wire (pts (xy 189.23 64.135) (xy 179.07 64.135))
     (stroke (width 0) (type default))
   )
+  (wire (pts (xy 14.605 149.225) (xy 17.145 149.225))
+    (stroke (width 0) (type default))
+  )
   (wire (pts (xy 256.54 130.81) (xy 256.54 139.7))
     (stroke (width 0) (type default))
@@
     (stroke (width 0) (type default))
   )
-  (wire (pts (xy 267.97 152.4) (xy 270.51 152.4))
+  (wire (pts (xy 257.81 151.13) (xy 255.27 151.13))
     (stroke (width 0) (type default))
   )
@@
   )
   (wire (pts (xy 201.93 33.655) (xy 201.93 36.195))
+    (stroke (width 0) (type default))
+  )
+  (wire (pts (xy 24.765 149.225) (xy 35.56 149.225))
     (stroke (width 0) (type default))
   )
@@
     (effects (font (size 1.27 1.27)) (justify left bottom))
   )
-  (label "~{SCLK_ENA}" (at 22.86 161.925 0) (fields_autoplaced)
-    (effects (font (size 1.27 1.27)) (justify left bottom))
+  (label "~{SCLK_ENA}" (at 86.36 80.645 180) (fields_autoplaced)
+    (effects (font (size 1.27 1.27)) (justify right bottom))
   )
   (label "A5" (at 179.07 53.975 0) (fields_autoplaced)
@@
     (effects (font (size 1.27 1.27)) (justify right bottom))
   )
-  (label "~{SCLK_ENA}" (at 245.11 149.86 0) (fields_autoplaced)
-    (effects (font (size 1.27 1.27)) (justify left bottom))
+  (label "~{SCLK_ENA}" (at 280.67 148.59 180) (fields_autoplaced)
+    (effects (font (size 1.27 1.27)) (justify right bottom))
   )
   (label "A2" (at 179.07 46.355 0) (fields_autoplaced)
@@
     )
   )
-  (symbol (lib_id "power:VCC") (at 270.51 144.78 0) (unit 1)
-    (in_bom yes) (on_board yes) (dnp no) (fields_autoplaced)
-    (property "Reference" "#PWR?" (at 270.51 148.59 0)
-      (effects (font (size 1.27 1.27)) hide)
-    )
-    (property "Value" "VCC" (at 270.51 139.7 0)
-      (effects (font (size 1.27 1.27)))
-    )
-    (property "Footprint" "" (at 270.51 144.78 0)
-      (effects (font (size 1.27 1.27)) hide)
-    )
-    (property "Datasheet" "" (at 270.51 144.78 0)
-      (effects (font (size 1.27 1.27)) hide)
-    )
-    (pin "1")
-    (instances
-      (project "fortuna-s"
-        (path "/01925f6f-51ef-4838-b51d-68dc0814d806"
-          (reference "#PWR?") (unit 1)
-        )
-      )
-      (project "fortuna-box"
-        (path "/0e4c4e8a-78e0-4f49-88dc-754c12656209/afd1b413-de30-4838-bb16-3d0c9f3cd196"
-          (reference "#PWR019") (unit 1)
-        )
-      )
-      (project "fortuna-5"
-        (path "/1f6368db-16b6-4786-887a-0cc62dc8c711"
-          (reference "#PWR02") (unit 1)
-        )
-      )
-    )
-  )
-  (symbol (lib_id "Switch:SW_DPDT_x2") (at 262.89 149.86 0) (unit 2)
-    (in_bom yes) (on_board yes) (dnp no) (fields_autoplaced)
-    (property "Reference" "SW1" (at 262.89 142.24 0)
-      (effects (font (size 1.27 1.27)))
-    )
-    (property "Value" "SW_DPDT_x2" (at 262.89 144.78 0)
-      (effects (font (size 1.27 1.27)))
-    )
-    (property "Footprint" "" (at 262.89 149.86 0)
-      (effects (font (size 1.27 1.27)) hide)
-    )
-    (property "Datasheet" "~" (at 262.89 149.86 0)
+  (symbol (lib_id "Switch:SW_DPDT_x2") (at 262.89 148.59 180) (unit 2)
+    (in_bom yes) (on_board yes) (dnp no)
+    (property "Reference" "SW1" (at 262.89 156.21 0)
+      (effects (font (size 1.27 1.27)))
+    )
+    (property "Value" "CLOCK" (at 262.89 153.67 0)
+      (effects (font (size 1.27 1.27)))
+    )
+    (property "Footprint" "" (at 262.89 148.59 0)
+      (effects (font (size 1.27 1.27)) hide)
+    )
+    (property "Datasheet" "~" (at 262.89 148.59 0)
       (effects (font (size 1.27 1.27)) hide)
     )
@@
     )
   )
+  (symbol (lib_id "Device:R") (at 14.605 156.21 0) (unit 1)
+    (in_bom yes) (on_board yes) (dnp no) (fields_autoplaced)
+    (property "Reference" "R1" (at 16.51 154.94 0)
+      (effects (font (size 1.27 1.27)) (justify left))
+    )
+    (property "Value" "R" (at 16.51 157.48 0)
+      (effects (font (size 1.27 1.27)) (justify left))
+    )
+    (property "Footprint" "" (at 12.827 156.21 90)
+      (effects (font (size 1.27 1.27)) hide)
+    )
+    (property "Datasheet" "~" (at 14.605 156.21 0)
+      (effects (font (size 1.27 1.27)) hide)
+    )
+    (pin "1")
+    (pin "2")
+    (instances
+      (project "fortuna-5"
+        (path "/1f6368db-16b6-4786-887a-0cc62dc8c711"
+          (reference "R1") (unit 1)
+        )
+      )
+    )
+  )
   (symbol (lib_id "power:VCC") (at 55.88 32.385 0) (unit 1)
     (in_bom yes) (on_board yes) (dnp no) (fields_autoplaced)
@@
     )
   )
-  (symbol (lib_id "Switch:SW_DPDT_x2") (at 261.62 128.27 0) (mirror y) (unit 1)
+  (symbol (lib_id "Switch:SW_DPDT_x2") (at 261.62 128.27 180) (unit 1)
     (in_bom yes) (on_board yes) (dnp no)
-    (property "Reference" "SW4" (at 261.62 120.65 0)
-      (effects (font (size 1.27 1.27)))
-    )
-    (property "Value" "SW_DPDT_x2" (at 261.62 123.19 0)
+    (property "Reference" "SW4" (at 261.62 135.89 0)
+      (effects (font (size 1.27 1.27)))
+    )
+    (property "Value" "CLOCK" (at 261.62 133.35 0)
       (effects (font (size 1.27 1.27)))
     )
@@
     )
   )
-  (symbol (lib_id "power:GND") (at 270.51 154.94 0) (unit 1)
-    (in_bom yes) (on_board yes) (dnp no) (fields_autoplaced)
-    (property "Reference" "#PWR?" (at 270.51 161.29 0)
-      (effects (font (size 1.27 1.27)) hide)
-    )
-    (property "Value" "GND" (at 270.51 160.02 0)
-      (effects (font (size 1.27 1.27)))
-    )
-    (property "Footprint" "" (at 270.51 154.94 0)
-      (effects (font (size 1.27 1.27)) hide)
-    )
-    (property "Datasheet" "" (at 270.51 154.94 0)
+  (symbol (lib_id "power:GND") (at 255.27 153.67 0) (mirror y) (unit 1)
+    (in_bom yes) (on_board yes) (dnp no) (fields_autoplaced)
+    (property "Reference" "#PWR?" (at 255.27 160.02 0)
+      (effects (font (size 1.27 1.27)) hide)
+    )
+    (property "Value" "GND" (at 255.27 158.75 0)
+      (effects (font (size 1.27 1.27)))
+    )
+    (property "Footprint" "" (at 255.27 153.67 0)
+      (effects (font (size 1.27 1.27)) hide)
+    )
+    (property "Datasheet" "" (at 255.27 153.67 0)
       (effects (font (size 1.27 1.27)) hide)
     )
@@
         )
       )
+    )
+  )
+  (symbol (lib_id "power:GND") (at 14.605 161.29 0) (unit 1)
+    (in_bom yes) (on_board yes) (dnp no) (fields_autoplaced)
+    (property "Reference" "#PWR?" (at 14.605 167.64 0)
+      (effects (font (size 1.27 1.27)) hide)
+    )
+    (property "Value" "GND" (at 14.605 166.37 0)
+      (effects (font (size 1.27 1.27)))
+    )
+    (property "Footprint" "" (at 14.605 161.29 0)
+      (effects (font (size 1.27 1.27)) hide)
+    )
+    (property "Datasheet" "" (at 14.605 161.29 0)
+      (effects (font (size 1.27 1.27)) hide)
+    )
+    (pin "1")
+    (instances
+      (project "fortuna-s"
+        (path "/01925f6f-51ef-4838-b51d-68dc0814d806"
+          (reference "#PWR?") (unit 1)
+        )
+      )
+      (project "fortuna-box"
+        (path "/0e4c4e8a-78e0-4f49-88dc-754c12656209/afd1b413-de30-4838-bb16-3d0c9f3cd196"
+          (reference "#PWR020") (unit 1)
+        )
+      )
+      (project "fortuna-5"
+        (path "/1f6368db-16b6-4786-887a-0cc62dc8c711"
+          (reference "#PWR02") (unit 1)
+        )
+      )
+    )
+  )
+  (symbol (lib_id "Device:LED") (at 20.955 149.225 0) (unit 1)
+    (in_bom yes) (on_board yes) (dnp no) (fields_autoplaced)
+    (property "Reference" "D2" (at 19.3675 143.51 0)
+      (effects (font (size 1.27 1.27)))
+    )
+    (property "Value" "CLOCK" (at 19.3675 146.05 0)
+      (effects (font (size 1.27 1.27)))
+    )
+    (property "Footprint" "" (at 20.955 149.225 0)
+      (effects (font (size 1.27 1.27)) hide)
+    )
+    (property "Datasheet" "~" (at 20.955 149.225 0)
+      (effects (font (size 1.27 1.27)) hide)
+    )
+    (pin "1")
+    (pin "2")
+    (instances
+      (project "fortuna-5"
+        (path "/1f6368db-16b6-4786-887a-0cc62dc8c711"
+          (reference "D2") (unit 1)
+        )
+      )

Commit message: .
Parts:
- added D3: INIT, symbol Device:LED
- added R3: R, symbol Device:R
Connections:
- net GND: now also R1.1, R3.1; no longer R1.2
- net at U1.F2 (PH4): now also D3.2 (A)
- net at D2.1 (K): now also R1.2; no longer R1.1
- new net: D3.1 (K), R3.2
Other:
- moved on the sheet: D2, R1
Changed lines of the file:
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@@
 (kicad_sch (version 20230121) (generator eeschema)
   (paper "A4")
+  (junction (at 15.24 149.225) (diameter 0) (color 0 0 0 0)
+  )
   (junction (at 191.77 132.08) (diameter 0) (color 0 0 0 0)
   )
@@
     (stroke (width 0) (type default))
   )
-  (wire (pts (xy 14.605 152.4) (xy 14.605 149.225))
-    (stroke (width 0) (type default))
-  )
   (wire (pts (xy -216.535 179.705) (xy -216.535 176.53))
     (stroke (width 0) (type default))
@@
     (stroke (width 0) (type default))
   )
+  (wire (pts (xy 24.765 144.145) (xy 27.94 144.145))
+    (stroke (width 0) (type default))
+  )
   (wire (pts (xy 153.67 55.245) (xy 163.83 55.245))
     (stroke (width 0) (type default))
@@
     (stroke (width 0) (type default))
   )
-  (wire (pts (xy 14.605 160.02) (xy 14.605 161.29))
+  (wire (pts (xy 15.24 149.225) (xy 15.24 153.035))
     (stroke (width 0) (type default))
   )
@@
     (stroke (width 0) (type default))
   )
+  (wire (pts (xy 17.145 144.145) (xy 15.24 144.145))
+    (stroke (width 0) (type default))
+  )
   (wire (pts (xy -117.475 153.67) (xy -128.27 153.67))
     (stroke (width 0) (type default))
@@
     (stroke (width 0) (type default))
   )
+  (wire (pts (xy 15.24 144.145) (xy 15.24 149.225))
+    (stroke (width 0) (type default))
+  )
   (wire (pts (xy 172.72 147.32) (xy 172.72 149.86))
     (stroke (width 0) (type default))
@@
     (stroke (width 0) (type default))
   )
-  (wire (pts (xy 14.605 149.225) (xy 17.145 149.225))
+  (wire (pts (xy 15.24 149.225) (xy 17.145 149.225))
     (stroke (width 0) (type default))
   )
@@
     (stroke (width 0) (type default))
   )
+  (wire (pts (xy 24.765 149.225) (xy 27.94 149.225))
+    (stroke (width 0) (type default))
+  )
   (wire (pts (xy -117.475 191.77) (xy -128.27 191.77))
     (stroke (width 0) (type default))
@@
   )
   (wire (pts (xy 201.93 33.655) (xy 201.93 36.195))
-    (stroke (width 0) (type default))
-  )
-  (wire (pts (xy 24.765 149.225) (xy 35.56 149.225))
     (stroke (width 0) (type default))
   )
@@
         (path "/1f6368db-16b6-4786-887a-0cc62dc8c711"
           (reference "U2") (unit 1)
+        )
+      )
+    )
+  )
+  (symbol (lib_id "Device:LED") (at 31.75 144.145 0) (unit 1)
+    (in_bom yes) (on_board yes) (dnp no)
+    (property "Reference" "D3" (at 28.575 142.875 0)
+      (effects (font (size 1.27 1.27)))
+    )
+    (property "Value" "INIT" (at 30.48 140.97 0)
+      (effects (font (size 1.27 1.27)))
+    )
+    (property "Footprint" "" (at 31.75 144.145 0)
+      (effects (font (size 1.27 1.27)) hide)
+    )
+    (property "Datasheet" "~" (at 31.75 144.145 0)
+      (effects (font (size 1.27 1.27)) hide)
+    )
+    (pin "1")
+    (pin "2")
+    (instances
+      (project "fortuna-5"
+        (path "/1f6368db-16b6-4786-887a-0cc62dc8c711"
+          (reference "D3") (unit 1)
         )
       )
@@
     )
   )
-  (symbol (lib_id "Device:R") (at 14.605 156.21 0) (unit 1)
-    (in_bom yes) (on_board yes) (dnp no) (fields_autoplaced)
-    (property "Reference" "R1" (at 16.51 154.94 0)
-      (effects (font (size 1.27 1.27)) (justify left))
-    )
-    (property "Value" "R" (at 16.51 157.48 0)
-      (effects (font (size 1.27 1.27)) (justify left))
-    )
-    (property "Footprint" "" (at 12.827 156.21 90)
-      (effects (font (size 1.27 1.27)) hide)
-    )
-    (property "Datasheet" "~" (at 14.605 156.21 0)
+  (symbol (lib_id "Device:R") (at 20.955 149.225 90) (unit 1)
+    (in_bom yes) (on_board yes) (dnp no)
+    (property "Reference" "R1" (at 20.955 151.765 90)
+      (effects (font (size 1.27 1.27)))
+    )
+    (property "Value" "R" (at 20.955 149.225 90)
+      (effects (font (size 1.27 1.27)))
+    )
+    (property "Footprint" "" (at 20.955 151.003 90)
+      (effects (font (size 1.27 1.27)) hide)
+    )
+    (property "Datasheet" "~" (at 20.955 149.225 0)
       (effects (font (size 1.27 1.27)) hide)
     )
@@
     )
   )
-  (symbol (lib_id "power:GND") (at 14.605 161.29 0) (unit 1)
-    (in_bom yes) (on_board yes) (dnp no) (fields_autoplaced)
-    (property "Reference" "#PWR?" (at 14.605 167.64 0)
-      (effects (font (size 1.27 1.27)) hide)
-    )
-    (property "Value" "GND" (at 14.605 166.37 0)
-      (effects (font (size 1.27 1.27)))
-    )
-    (property "Footprint" "" (at 14.605 161.29 0)
-      (effects (font (size 1.27 1.27)) hide)
-    )
-    (property "Datasheet" "" (at 14.605 161.29 0)
+  (symbol (lib_id "power:GND") (at 15.24 153.035 0) (unit 1)
+    (in_bom yes) (on_board yes) (dnp no)
+    (property "Reference" "#PWR?" (at 15.24 159.385 0)
+      (effects (font (size 1.27 1.27)) hide)
+    )
+    (property "Value" "GND" (at 15.24 156.845 0)
+      (effects (font (size 1.27 1.27)))
+    )
+    (property "Footprint" "" (at 15.24 153.035 0)
+      (effects (font (size 1.27 1.27)) hide)
+    )
+    (property "Datasheet" "" (at 15.24 153.035 0)
       (effects (font (size 1.27 1.27)) hide)
     )
@@
     )
   )
-  (symbol (lib_id "Device:LED") (at 20.955 149.225 0) (unit 1)
-    (in_bom yes) (on_board yes) (dnp no) (fields_autoplaced)
-    (property "Reference" "D2" (at 19.3675 143.51 0)
-      (effects (font (size 1.27 1.27)))
-    )
-    (property "Value" "CLOCK" (at 19.3675 146.05 0)
-      (effects (font (size 1.27 1.27)))
-    )
-    (property "Footprint" "" (at 20.955 149.225 0)
-      (effects (font (size 1.27 1.27)) hide)
-    )
-    (property "Datasheet" "~" (at 20.955 149.225 0)
+  (symbol (lib_id "Device:LED") (at 31.75 149.225 0) (unit 1)
+    (in_bom yes) (on_board yes) (dnp no)
+    (property "Reference" "D2" (at 27.94 147.955 0)
+      (effects (font (size 1.27 1.27)))
+    )
+    (property "Value" "CLOCK" (at 31.115 152.4 0)
+      (effects (font (size 1.27 1.27)))
+    )
+    (property "Footprint" "" (at 31.75 149.225 0)
+      (effects (font (size 1.27 1.27)) hide)
+    )
+    (property "Datasheet" "~" (at 31.75 149.225 0)
       (effects (font (size 1.27 1.27)) hide)
     )
@@
         )
       )
+    )
+  )
+  (symbol (lib_id "Device:R") (at 20.955 144.145 90) (unit 1)
+    (in_bom yes) (on_board yes) (dnp no)
+    (property "Reference" "R3" (at 20.955 146.685 90)
+      (effects (font (size 1.27 1.27)))
+    )
+    (property "Value" "R" (at 20.955 144.145 90)
+      (effects (font (size 1.27 1.27)))
+    )
+    (property "Footprint" "" (at 20.955 145.923 90)
+      (effects (font (size 1.27 1.27)) hide)
+    )
+    (property "Datasheet" "~" (at 20.955 144.145 0)
+      (effects (font (size 1.27 1.27)) hide)
+    )
+    (pin "1")
+    (pin "2")
+    (instances
+      (project "fortuna-5"
+        (path "/1f6368db-16b6-4786-887a-0cc62dc8c711"
+          (reference "R3") (unit 1)
+        )
+      )
