File: circuit/fortuna-5.kicad_sch (KiCad schematic)
At the start: 17 parts, among them J8 USB-C Power, SW1 SW_Push, SW4 CLOCK, U1 ATmega2560-16C, U2 Z80CPU, U3 AS6C4008-55PCN, U4 74HC04, U5 74LS32, U6 74HC00

Commit message: .
Parts:
- added J1: Debug, symbol Connector_Generic:Conn_01x06
Connections:
- net GND: now also J1.1 (Pin_1)
- net RX: now also U1.F8 (PJ0), J1.5 (Pin_5)
- net TX: now also U1.F7 (PJ1), J1.4 (Pin_4)
- net ~{CWAIT}: now also U1.E3 (PH1); no longer U1.F8 (PJ0)
Changed lines of the file:
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@@
+    (stroke (width 0) (type default))
+  )
+  (wire (pts (xy 130.81 162.56) (xy 130.81 146.685))
     (stroke (width 0) (type default))
   )
@@
     (stroke (width 0) (type default))
   )
+  (wire (pts (xy 138.43 154.305) (xy 128.27 154.305))
+    (stroke (width 0) (type default))
+  )
   (wire (pts (xy -205.105 158.75) (xy -194.31 158.75))
     (stroke (width 0) (type default))
@@
     (stroke (width 0) (type default))
   )
+  (wire (pts (xy 130.81 146.685) (xy 128.27 146.685))
+    (stroke (width 0) (type default))
+  )
   (wire (pts (xy 172.72 132.08) (xy 172.72 134.62))
     (stroke (width 0) (type default))
@@
     (stroke (width 0) (type default))
   )
+  (wire (pts (xy 138.43 156.845) (xy 128.27 156.845))
+    (stroke (width 0) (type default))
+  )
   (wire (pts (xy 189.23 43.815) (xy 179.07 43.815))
     (stroke (width 0) (type default))
@@
     (stroke (width 0) (type default))
   )
+  (wire (pts (xy 25.4 113.665) (xy 35.56 113.665))
+    (stroke (width 0) (type default))
+  )
   (wire (pts (xy 76.2 65.405) (xy 86.36 65.405))
     (stroke (width 0) (type default))
   )
+  (wire (pts (xy 35.56 136.525) (xy 25.4 136.525))
+    (stroke (width 0) (type default))
+  )
   (wire (pts (xy 189.23 84.455) (xy 179.07 84.455))
     (stroke (width 0) (type default))
@@
     (stroke (width 0) (type default))
   )
+  (wire (pts (xy 25.4 111.125) (xy 35.56 111.125))
+    (stroke (width 0) (type default))
+  )
   (wire (pts (xy 35.56 106.045) (xy 25.4 106.045))
     (stroke (width 0) (type default))
@@
   )
   (wire (pts (xy 189.23 46.355) (xy 179.07 46.355))
-    (stroke (width 0) (type default))
-  )
-  (wire (pts (xy 35.56 111.125) (xy 25.4 111.125))
     (stroke (width 0) (type default))
   )
@@
     (effects (font (size 1.27 1.27)) (justify left bottom))
   )
+  (label "TX" (at 138.43 154.305 180) (fields_autoplaced)
+    (effects (font (size 1.27 1.27)) (justify right bottom))
+  )
   (label "A7" (at 163.83 60.325 180) (fields_autoplaced)
     (effects (font (size 1.27 1.27)) (justify right bottom))
@@
     (effects (font (size 1.27 1.27)) (justify right bottom))
   )
+  (label "~{CWAIT}" (at 25.4 136.525 0) (fields_autoplaced)
+    (effects (font (size 1.27 1.27)) (justify left bottom))
+  )
   (label "A1" (at 163.83 45.085 180) (fields_autoplaced)
     (effects (font (size 1.27 1.27)) (justify right bottom))
@@
     (effects (font (size 1.27 1.27)) (justify left bottom))
   )
+  (label "RX" (at 138.43 156.845 180) (fields_autoplaced)
+    (effects (font (size 1.27 1.27)) (justify right bottom))
+  )
   (label "~{ROM_WE}" (at -117.475 128.27 180) (fields_autoplaced)
     (effects (font (size 1.27 1.27)) (justify right bottom))
@@
     (effects (font (size 1.27 1.27)) (justify right bottom))
   )
+  (label "RX" (at 25.4 111.125 0) (fields_autoplaced)
+    (effects (font (size 1.27 1.27)) (justify left bottom))
+  )
   (label "~{M1}" (at -117.475 196.85 180) (fields_autoplaced)
     (effects (font (size 1.27 1.27)) (justify right bottom))
@@
     (effects (font (size 1.27 1.27)) (justify right bottom))
   )
+  (label "TX" (at 25.4 113.665 0) (fields_autoplaced)
+    (effects (font (size 1.27 1.27)) (justify left bottom))
+  )
   (label "~{CS1}" (at 86.36 75.565 180) (fields_autoplaced)
     (effects (font (size 1.27 1.27)) (justify right bottom))
@@
   (label "~{IORQ}" (at 86.36 111.125 180) (fields_autoplaced)
     (effects (font (size 1.27 1.27)) (justify right bottom))
-  )
-  (label "~{CWAIT}" (at 25.4 111.125 0) (fields_autoplaced)
-    (effects (font (size 1.27 1.27)) (justify left bottom))
   )
   (label "D1" (at 86.36 45.085 180) (fields_autoplaced)
@@
         (path "/1f6368db-16b6-4786-887a-0cc62dc8c711"
           (reference "U2") (unit 1)
+        )
+      )
+    )
+  )
+  (symbol (lib_id "Connector_Generic:Conn_01x06") (at 123.19 151.765 0) (mirror y) (unit 1)
+    (in_bom yes) (on_board yes) (dnp no) (fields_autoplaced)
+    (property "Reference" "J1" (at 123.19 140.97 0)
+      (effects (font (size 1.27 1.27)))
+    )
+    (property "Value" "Debug" (at 123.19 143.51 0)
+      (effects (font (size 1.27 1.27)))
+    )
+    (property "Footprint" "" (at 123.19 151.765 0)
+      (effects (font (size 1.27 1.27)) hide)
+    )
+    (property "Datasheet" "~" (at 123.19 151.765 0)
+      (effects (font (size 1.27 1.27)) hide)
+    )
+    (pin "1")
+    (pin "2")
+    (pin "3")
+    (pin "4")
+    (pin "5")
+    (pin "6")
+    (instances
+      (project "fortuna-5"
+        (path "/1f6368db-16b6-4786-887a-0cc62dc8c711"
+          (reference "J1") (unit 1)
         )
       )
@@
         )
       )
+    )
+  )
+  (symbol (lib_id "power:GND") (at 130.81 162.56 0) (unit 1)
+    (in_bom yes) (on_board yes) (dnp no) (fields_autoplaced)
+    (property "Reference" "#PWR?" (at 130.81 168.91 0)
+      (effects (font (size 1.27 1.27)) hide)
+    )
+    (property "Value" "GND" (at 130.81 167.64 0)
+      (effects (font (size 1.27 1.27)))
+    )
+    (property "Footprint" "" (at 130.81 162.56 0)
+      (effects (font (size 1.27 1.27)) hide)
+    )
+    (property "Datasheet" "" (at 130.81 162.56 0)
+      (effects (font (size 1.27 1.27)) hide)
+    )
+    (pin "1")
+    (instances
+      (project "fortuna-s"
+        (path "/01925f6f-51ef-4838-b51d-68dc0814d806"
+          (reference "#PWR?") (unit 1)
+        )
+      )
+      (project "fortuna-box"
+        (path "/0e4c4e8a-78e0-4f49-88dc-754c12656209/afd1b413-de30-4838-bb16-3d0c9f3cd196"
+          (reference "#PWR020") (unit 1)
+        )
+      )
+      (project "fortuna-5"
+        (path "/1f6368db-16b6-4786-887a-0cc62dc8c711"
+          (reference "#PWR016") (unit 1)
+        )
+      )

Commit message: .
Parts:
- removed D6: LED, symbol Device:LED
- removed J8: USB-C Power, symbol Connector:USB_C_Receptacle_PowerOnly_6P
- removed R17: 220, symbol Device:R
- removed X?: 20 Mhz, Oscillator:Oscillator_DIP-14, symbol Oscillator:ACO-xxxMHz
- added C1, C2: C, symbol Device:C
- added R4: 1M, symbol Device:R
- added U7: 74HC14, symbol 74xx:74HC14
- added Y1: 20Mhz, symbol Device:Crystal
Connections:
- net GND: now also C1.2, C2.2
- net at SW4.3 (C): now also U7.8
- new net: U7.4, U7.5
- new net: U7.6, U7.9
- new net: C2.1, R4.2, U7.2, U7.3, Y1.2
- new net: C1.1, R4.1, U7.1, Y1.1
- no-connect marks 27 -> 25
Other:
- note removed: "POWER"
- moved on the sheet: J1, SW1B, SW4A, U4A, U5A, U6A, U6B, U6C, U6D

Commit message: .
Parts:
- added J2: Conn_01x08, symbol Connector_Generic:Conn_01x08
Connections:
- net GND: now also J2.6 (Pin_6)
- net MISO: now also J2.4 (Pin_4)
- net MOSI: now also J2.3 (Pin_3)
- net SCK: now also J2.5 (Pin_5)
- net VCC: now also J2.7 (Pin_7)
- net ~{SD_CD}: now reaches U1.D1 (PE3)
- net ~{SD_CD}: now also J2.1 (Pin_1)
- net ~{SD_CS}: now reaches U1.K1 (PB7)
- net ~{SD_CS}: now also J2.2 (Pin_2)
- no-connect marks 25 -> 29
Other:
- note added: "Debug"
- note added: "SDCard"
- moved on the sheet: U4A, U5A, U6A, U6B, U6C, U6D
