File: circuit/fortuna-5.kicad_sch (KiCad schematic)
At the start: 20 parts, among them J1 Debug, J2 Conn_01x08, SW1 SW_Push, SW4 CLOCK, U1 ATmega2560-16C, U2 Z80CPU, U3 AS6C4008-55PCN, U4 74HC04, U5 74LS32, U6 74HC00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

Commit message: .
Parts:
- added J3: ~, symbol Connector_Generic:Conn_02x05_Counter_Clockwise
Connections:
- net ~{CS0} is gone; now on net ~{SD_CS}: U1.F4 (PB0)
- net GND: now also J3.5 (Pin_5)
- net MISO: now also J3.3 (Pin_3)
- net MOSI: now also J3.2 (Pin_2)
- net RX: now also J3.10 (Pin_10)
- net SCK: now also J3.4 (Pin_4)
- net TX: now also J3.9 (Pin_9)
- net VCC: now also J3.1 (Pin_1)
- net ~{CS1}: now also J3.8 (Pin_8)
- net ~{CS2}: now also J3.7 (Pin_7)
- net ~{INT}: now also J3.6 (Pin_6)
- net ~{SD_CS}: no longer U1.K1 (PB7)
Other:
- note added: "External SPI"

Commit message: .
Other:
- note added: "NOTCH->"
Changed lines of the file:
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@@
     (effects (font (size 3 3) (thickness 0.6) bold) (justify left bottom))
+  )
+  (text "NOTCH->" (at 177.165 123.19 0)
+    (effects (font (size 1.27 1.27)) (justify left bottom))
   )
   (text "External SPI" (at 189.865 111.125 0)
